File: PC-SPRINT v2/PC-SPRINT.sch (KiCad schematic (older format))
At the start: 16 parts, among them J1 TB1, U1 8284A, U2 8284A, U3 8284A, X1 22.11 MHz

Commit message: Added PC-SPRINT v2 information and files
Parts:
- added D3, D4, D5, D6: 1N4148, Diode_THT:D_DO-35_SOD27_P7.62mm_Horizontal, symbol PC-SPRINT-rescue:D
- added J2: DMA1, Connector_PinSocket_2.54mm:PinSocket_1x02_P2.54mm_Vertical, symbol Connector_Generic:Conn_01x02
- added Q1: Q_NPN_BCE, TO_SOT_Packages_THT:TO-92_Molded_Wide_Oval, symbol Device:Q_NPN_BCE
- added R6, R7, R8: 10K, Resistor_THT:R_Axial_DIN0204_L3.6mm_D1.6mm_P7.62mm_Horizontal, symbol PC-SPRINT-rescue:R
- added R9: 3.3K, Resistor_THT:R_Axial_DIN0204_L3.6mm_D1.6mm_P7.62mm_Horizontal, symbol PC-SPRINT-rescue:R
- C1, C3, C4: footprint Capacitors_THT:CP_Radial_Tantal_D4.5mm_P2.50mm -> Capacitor_THT:CP_Radial_Tantal_D4.5mm_P2.50mm; symbol CP -> PC-SPRINT-rescue:CP
- C2: footprint Capacitors_THT:C_Disc_D5.0mm_W2.5mm_P2.50mm -> Capacitor_THT:C_Disc_D5.0mm_W2.5mm_P2.50mm; symbol C -> PC-SPRINT-rescue:C
- D1, D2: footprint Diodes_THT:D_DO-35_SOD27_P7.62mm_Horizontal -> Diode_THT:D_DO-35_SOD27_P7.62mm_Horizontal; symbol D -> PC-SPRINT-rescue:D
- J1: footprint Pin_Headers:Pin_Header_Straight_1x04_Pitch2.54mm -> Connector_PinSocket_2.54mm:PinSocket_1x04_P2.54mm_Vertical; symbol Conn_01x04 -> Connector_Generic:Conn_01x04
- R1, R2, R3, R4, R5: footprint Resistors_THT:R_Axial_DIN0204_L3.6mm_D1.6mm_P7.62mm_Horizontal -> Resistor_THT:R_Axial_DIN0204_L3.6mm_D1.6mm_P7.62mm_Horizontal; symbol R -> PC-SPRINT-rescue:R
- U1, U2, U3: footprint Housings_DIP:DIP-18_W7.62mm_LongPads -> Package_DIP:DIP-18_W7.62mm_LongPads; symbol 8284A -> PC-SPRINT-rescue:8284A
- X1: footprint Crystals:Crystal_HC18-U_Vertical -> Crystal:Crystal_HC18-U_Vertical; symbol Crystal -> PC-SPRINT-rescue:Crystal
Connections:
- net at C1.1, C2.1, R3.1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: now also R8.1, R9.1
- net at C1.2, C2.2, C3.2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: now also Q1.3 (E), R6.1
- net at C3.1, J1.1 (Pin_1), R5.2: now also D5.1 (K); no longer U3.11 (~RES)
- new net: D5.2 (A), D6.2 (A), R9.2, U3.11 (~RES)
- new net: D4.1 (K), J2.1 (Pin_1)
- new net: D3.1 (K), J2.2 (Pin_2)
- new net: D3.2 (A), D4.2 (A), R6.2, R7.2
- new net: Q1.1 (B), R7.1
- new net: D6.1 (K), Q1.2 (C), R8.2
